File: KiCad_Traffic_Light_Controller_demo/KiCad_Traffic_Light_Controller_demo.kicad_sch (KiCad schematic)
At the start: 40 parts, among them J1 Conn_02x08_Odd_Even, J2 Conn_02x08_Odd_Even, U1 SM420561N, U2 SM420561N

Commit message: Updated KiCad Files
Parts:
- added C1, C4: C_Polarized_Small, symbol Device:C_Polarized_Small
- added C2, C3, C5: 0.22u, symbol Device:C_Small
- added D11, D12, D13: 1N4148W, Diode_SMD:D_SOD-123, symbol Diode:1N4148W
- added H1, H2, H3, H4: MountingHole, symbol Mechanical:MountingHole
- added J3: Conn_02x05_Odd_Even, symbol Connector_Generic:Conn_02x05_Odd_Even
- added J4: +5V, symbol Connector:Screw_Terminal_01x02
- added R27, R28, R29, R30, R31, R32: 47K, symbol Device:R
- added SW1: RST, symbol Switch:SW_Push
- added SW2: OVR, symbol Switch:SW_SPDT
- added SW3: EN, symbol Switch:SW_SPDT
- added U3: LM1117DT-3.3, Package_TO_SOT_SMD:TO-252-3_TabPin2, symbol Regulator_Linear:LM1117DT-3.3
Connections:
- net +3.3V: now also C4.1, R27.2, R30.2, R32.2, U3.2 (VO)
- net GND: now also C1.2, C2.2, C3.2, C4.2, C5.2, J3.10 (Pin_10), J3.2 (Pin_2), J3.4 (Pin_4), J3.6 (Pin_6), J3.8 (Pin_8), J4.2 (Pin_2), SW1.1, SW2.3 (C), SW3.3 (C), U3.1 (GND)
- new net: D13.2 (A), R31.1, R32.1, SW3.2 (B)
- new net: D11.2 (A), R28.1, R30.1, SW2.2 (B)
- new net: D12.2 (A), R27.1, R29.2, SW1.2
- new net +5V: C1.1, J3.7 (Pin_7), J3.9 (Pin_9), J4.1 (Pin_1), U3.3 (VI)
- new net EN: C5.1, D13.1 (K), J3.3 (Pin_3), R31.2
- new net OVR: C2.1, D11.1 (K), J3.5 (Pin_5), R28.2
- new net RST: C3.1, D12.1 (K), J3.1 (Pin_1), R29.1
- no-connect marks 0 -> 2
Other:
- note added: "+3.3V VOLTAGE REGULATOR"
- note added: "EMERGENCY OVERRIDE"
- note added: "ENABLE"
- note added: "MOUNTING HOLES"
- note added: "RESET"
- moved on the sheet: D1, D10, D2, D3, D4, D5, D6, D7, D8, D9, J1, J2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

Commit message: Updated KiCad_Traffic_Light_Controller_demo
Parts:
- removed C1, C4: C_Polarized_Small, symbol Device:C_Polarized_Small
- removed C2, C3, C5: 0.22u, symbol Device:C_Small
- added C1, C4: 10u, symbol Device:C_Polarized
- added C2, C3, C5: 0.22u, symbol Device:C
Connections:
- net EW_HEX_H is gone; now on net EW_HEX_G: R15.1
- net NS_HEX_H is gone; now on net NS_HEX_G: R7.1
- net +3.3V: now also C4.1
- net +5V: now also J4.2 (Pin_2), C1.1; no longer J4.1 (Pin_1)
- net EN: now also C5.1
- net EWC_GRN: now also D4.2 (A)
- net EWC_RED: now also D6.2 (A)
- net EWC_YLW: now also D5.2 (A)
- net EWP_GRN: now also D9.2 (A)
- net EWP_RED: now also D10.2 (A)
- net EW_HEX_E: now also R13.1
- net EW_HEX_F: now also R14.1; no longer R13.1
- net EW_HEX_G: no longer R14.1
- net GND: now also J4.1 (Pin_1), C1.2, C2.2, C3.2, C4.2, C5.2; no longer J4.2 (Pin_2)
- net NSC_GRN: no longer D4.2 (A)
- net NSC_RED: no longer D6.2 (A)
- net NSC_YLW: no longer D5.2 (A)
- net NSP_GRN: no longer D9.2 (A)
- net NSP_RED: no longer D10.2 (A)
- net NS_HEX_E: now also R5.1
- net NS_HEX_F: now also R6.1; no longer R5.1
- net NS_HEX_G: no longer R6.1
- net OVR: now also C2.1
- net RST: now also C3.1
Other:
- note added: "CONTROL LOGIC"
- moved on the sheet: D1, D10, D11, D12, D2, D3, D4, D5, D6, D7, D8, D9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

Commit message: Updated KiCad_Traffic_Light_Controller_demo
Parts:
- removed C1, C4: 10u, symbol Device:C_Polarized
- removed C2, C3, C5: 0.22u, symbol Device:C
- removed R1, R10, R11, R12, R13, R14, R15, R16, R17, R18, R19, R2, R20, R21, R22, R23, R24, R25, R26, R3, R4, R5, R6, R7, R8, R9: 130R, symbol Device:R
- removed R27, R28, R29, R30, R31, R32: 47K, symbol Device:R
- added C1: 10u, symbol Device:C_Polarized_Small
- added C2, C3, C5: 0.22u, symbol Device:C_Small
- added C4: 100u, symbol Device:C_Polarized_Small
- added R1, R10, R11, R12, R13, R14, R15, R16, R17, R18, R19, R2, R20, R21, R22, R23, R24, R25, R26, R27, R28, R29, R3, R30, R31, R32, R4, R5, R6, R7, R8, R9: 130R, symbol Device:R_Small
Connections:
- net +3.3V: now also C4.1, R27.2, R30.1, R32.2
- net +5V: now also C1.1
- net EN: now also C5.1, R31.2
- net EW_HEX_A: now also R9.1
- net EW_HEX_B: now also R10.1
- net EW_HEX_C: now also R11.1
- net EW_HEX_D: now also R12.1
- net EW_HEX_DP: now also R16.1
- net EW_HEX_E: now also R13.1
- net EW_HEX_F: now also R14.1
- net EW_HEX_G: now also R15.1
- net GND: now also C1.2, C2.2, C3.2, C4.2, C5.2, R17.1, R18.1, R19.1, R20.1, R21.1, R22.1, R23.1, R24.1, R25.1, R26.1
- net NS_HEX_A: now also R1.1
- net NS_HEX_B: now also R2.1
- net NS_HEX_C: now also R3.1
- net NS_HEX_D: now also R4.1
- net NS_HEX_DP: now also R8.1
- net NS_HEX_E: now also R5.1
- net NS_HEX_F: now also R6.1
- net NS_HEX_G: now also R7.1
- net OVR: now also C2.1, R28.1
- net RST: now also C3.1, R29.1
- net at D2.1 (K): now also R18.2
- net at D8.1 (K): now also R24.2
- net at D13.2 (A), SW3.2 (B): now also R31.1, R32.1
- net at D1.1 (K): now also R17.2
- net at D11.2 (A), SW2.2 (B): now also R28.2, R30.2
- net at U2.2 (D): now also R12.2
- net at D12.2 (A), SW1.2: now also R27.1, R29.2
- net at D7.1 (K): now also R23.2
- net at D4.1 (K): now also R20.2
- net at D9.1 (K): now also R25.2
- net at U2.6 (B): now also R10.2
- net at U1.5 (DP): now also R8.2
- net at U2.5 (DP): now also R16.2
- net at D3.1 (K): now also R19.2
- net at D10.1 (K): now also R26.2
- net at U1.1 (E): now also R5.2
- net at U1.10 (G): now also R7.2
- net at U1.2 (D): now also R4.2
- net at U1.4 (C): now also R3.2
- net at U1.6 (B): now also R2.2
- net at U1.7 (A): now also R1.2
- net at U1.9 (F): now also R6.2
- net at U2.7 (A): now also R9.2
- net at U2.10 (G): now also R15.2
- net at D6.1 (K): now also R22.2
- net at U2.4 (C): now also R11.2
- net at U2.1 (E): now also R13.2
- net at U2.9 (F): now also R14.2
- net at D5.1 (K): now also R21.2
Other:
- moved on the sheet: D1, D10, D2, D3, D7, D8, D9, J3, J4, SW1

Commit message: Updated KiCad_Traffic_Light_Controller_demo file
Parts:
- C1: footprint (none) -> Capacitor_SMD:CP_Elec_4x5.3
- C2, C3, C5: footprint (none) -> Capacitor_SMD:C_1206_3216Metric_Pad1.33x1.80mm_HandSolder
- C4: footprint (none) -> Capacitor_SMD:CP_Elec_6.3x5.8
- D1, D10, D2, D3, D4, D5, D6, D7, D8, D9: footprint (none) -> LED_THT:LED_D5.0mm
- H1, H2, H3, H4: footprint (none) -> MountingHole:MountingHole_2.2mm_M2
- J1, J2: footprint (none) -> Connector_PinHeader_2.54mm:PinHeader_2x08_P2.54mm_Vertical
- J3: footprint (none) -> Connector_PinHeader_2.54mm:PinHeader_2x05_P2.54mm_Vertical
- J4: footprint (none) -> my_footprints:Terminal_Block_5mm
- R1, R10, R11, R12, R13, R14, R15, R16, R17, R18, R19, R2, R20, R21, R22, R23, R24, R25, R26, R3, R4, R5, R6, R7, R8, R9: footprint (none) -> Resistor_SMD:R_1206_3216Metric_Pad1.30x1.75mm_HandSolder
- R27, R28, R29, R30, R31, R32: value 130R -> 47K; footprint (none) -> Resistor_SMD:R_1206_3216Metric_Pad1.30x1.75mm_HandSolder
- SW1: footprint (none) -> my_footprints:tact_switch_5mm
- SW2, SW3: footprint (none) -> my_footprints:slide_switch_2.54mm
- U3: footprint Package_TO_SOT_SMD:TO-252-3_TabPin2 -> Package_TO_SOT_SMD:SOT-223
